Commit message: changed parameters

File: exporttest.urdf (robot description, URDF)
Before this commit: robot cube.urdf, 1 links, 0 joints
Links:
- link baseLink: geometry collision mesh filename=unityexport.obj scale=0.2 0.2 0.2; visual mesh filename=unityexport.obj scale=0.2 0.2 0.2

Commit message: added mesh for testing and made changes to noise

File: exporttest.urdf (robot description, URDF)
Before this commit: robot cube.urdf, 1 links, 0 joints
Links:
- link baseLink: geometry collision mesh filename=meshEXPORT.obj scale=0.2 0.2 0.2; visual mesh filename=meshEXPORT.obj scale=0.2 0.2 0.2
