Commit message: fixed scaling and cleaned up

File: PybulletFiles/exporttest.urdf (robot description, URDF)
Before this commit: robot cube.urdf, 1 links, 0 joints
Links:
- link baseLink: geometry collision mesh filename=unityexport.obj scale=0.04 0.04 0.04; visual mesh filename=unityexport.obj scale=0.04 0.04 0.04
